File: crates/hauksbee-extract/tests/fixtures/eagle_ties/declared.sch (EAGLE design)
At the start: 0 parts

Commit message: Fix Eagle schematic net-tie parity
Require physical vertical copper and canonical pin/net identity before qualifying Eagle contacts. Preserve the established APIs while carrying optional schematic evidence through CLI, TUI, reports, standalone web analysis, and live launch.
Parts:
- added R1: 10k, device:R
Connections:
- new net AGND: R1.2
- new net GND: R1.1
Changed lines of the file:
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@@
 <?xml version="1.0"?>
 <eagle version="6.6.0"><drawing><schematic>
-<parts><part name="SUPPLY1" library="supply1" library_urn="urn:adsk.eagle:library:1" deviceset="GND"/><part name="AGND1" library="supply1" library_urn="urn:adsk.eagle:library:1" deviceset="AGND"/></parts>
-<sheets><sheet><nets><net name="GND"><segment><pinref part="SUPPLY1"/><pinref part="AGND1"/></segment></net></nets></sheet></sheets>
+<parts><part name="SUPPLY1" library="supply1" library_urn="urn:adsk.eagle:library:1" deviceset="GND"/><part name="AGND1" library="supply1" library_urn="urn:adsk.eagle:library:1" deviceset="AGND"/><part name="R1" library="device" deviceset="R" device="" value="10k"/></parts>
+<sheets><sheet><nets><net name="GND"><segment><pinref part="SUPPLY1"/><pinref part="AGND1"/><pinref part="R1" gate="G$1" pin="1"/></segment></net><net name="AGND"><segment><pinref part="R1" gate="G$1" pin="2"/></segment></net></nets></sheet></sheets>
 </schematic></drawing></eagle>
